Commit message: 4 standoff rods added to barista_robot_model.urdf.

File: urdf/barista_robot_model.urdf (robot description, URDF)
Before this commit: robot barista_robot, 9 links, 8 joints
Links:
- added link standoff_rod_1, mass 0.05; collision cylinder length=0.26 radius=0.01; visual cylinder length=0.26 radius=0.01
- added link standoff_rod_2, mass 0.05; collision cylinder length=0.26 radius=0.01; visual cylinder length=0.26 radius=0.01
- added link standoff_rod_3, mass 0.05; collision cylinder length=0.26 radius=0.01; visual cylinder length=0.26 radius=0.01
- added link standoff_rod_4, mass 0.05; collision cylinder length=0.26 radius=0.01; visual cylinder length=0.26 radius=0.01
Joints:
- added joint base_to_standoff_rod_1: type fixed, parent base_link, child standoff_rod_1, origin xyz=0.05 0.138 0.165 rpy=0 0 0
- added joint base_to_standoff_rod_2: type fixed, parent base_link, child standoff_rod_2, origin xyz=-0.05 0.138 0.165 rpy=0 0 0
- added joint base_to_standoff_rod_3: type fixed, parent base_link, child standoff_rod_3, origin xyz=0.05 -0.138 0.165 rpy=0 0 0
- added joint base_to_standoff_rod_4: type fixed, parent base_link, child standoff_rod_4, origin xyz=-0.05 -0.138 0.165 rpy=0 0 0

Commit message: Added: laser_scan_link with meshes and laser_scan_joint to baselink. Tested  visualization works on rviz.

File: urdf/barista_robot_model.urdf (robot description, URDF)
Before this commit: robot barista_robot, 13 links, 12 joints
Links:
- added link laser_scan_link, mass 0.01; collision cylinder length=0.0408 radius=0.037493; visual mesh filename=package://barista_robot_description/meshes/lidar/rplidar.dae scale=1.0 1.0 1.0
Joints:
- added joint laser_scan_joint: type continuous, parent base_link, child laser_scan_link, origin xyz=0.103 0 0.0775 rpy=0 0 0, axis 0 0 1, limit effort=10.0 velocity=2.0

Commit message: Added improved laser_scan_link and joint. Laser now shows in both rviz and gazebo. Updated barista_urdf.launch.py to work correctly with gazebo. Fixed the bug where gazebo could not find the laser meshes. Added gazebo_ros, robot_state_publisher and joint_state_publisher to both package.xml and CMakeLists.txt. Created a new subfolder under /meshes to group all 2D lidars in /LIDAR_2D_Sensor. Added multiple 2D Lidar .dae files, meshes, into /LIDAR_2D_Sensor. Added README.md into /LIDAR_2D_Sensor, to show the source of the LIDAR meshes.

File: urdf/barista_robot_model.urdf (robot description, URDF)
Before this commit: robot barista_robot, 14 links, 13 joints
Links:
- link back_roll_link: mass 0.001 -> 0.005; geometry collision cylinder length=0.001 radius=0.0145; visual cylinder length=0.001 radius=0.0145
- link back_yaw_link: mass 0.01 -> 0.005; geometry collision cylinder length=0.001 radius=0.0145; visual cylinder length=0.001 radius=0.0145
- link front_pitch_link: geometry collision sphere radius=0.03; visual sphere radius=0.03
- link front_roll_link: mass 0.01 -> 0.005
- link front_yaw_link: mass 0.01 -> 0.005
- link laser_scan_link: geometry collision cylinder length=0.0408 radius=0.037493; visual mesh filename=package://barista_robot_description/meshes/LIDAR_2D_Sensor/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 scale=1.0 1.0 1.0
Joints:
- joint laser_scan_joint: axis 0 0 1 -> (none); limit effort=10.0 velocity=2.0 -> (none); origin xyz=0.103 0 0.0775 rpy=0 0 0 -> xyz=0 0 0.0775 rpy=0 0 0; type continuous -> fixed

Commit message: Added a new link and frame: laser_scan_frame_link and laser_scan_frame_joint for positioning correctly the Gazebo laser sensor.Added Gazebo laser plugin. Tested on both Rviz and Gazebo. This Gazebo sensor laser plugin is publishing the scans to /barista_robot/scan topic successfully.

File: urdf/barista_robot_model.urdf (robot description, URDF)
Before this commit: robot barista_robot, 14 links, 13 joints
Links:
- added link laser_scan_frame_link
Joints:
- removed joint laser_scan_joint
- added joint laser_scan_frame_joint: type fixed, parent laser_scan_link, child laser_scan_frame_link, origin xyz=0 0 0.0306 rpy=0 0 0
- added joint laser_scan_link_joint: type fixed, parent base_link, child laser_scan_link, origin xyz=0 0 0.0775 rpy=0 0 0

Commit message: Changed the mass of laser_scan_link from 0.01 to 0.2 and recalculated the inertias. Updated the update rate of laser sensor from 10.0 to 30.0. Changed the sensor name from laser_sensor to sensor_ray.

File: urdf/barista_robot_model.urdf (robot description, URDF)
Before this commit: robot barista_robot, 15 links, 14 joints
Links:
- link laser_scan_link: mass 0.01 -> 0.20

Commit message: Adjusted wheel sizes and caster wheel sizes, recalculated inertia. Created new urdf_vis.rviz save file. The barista robot works now with /cmd_vel, /odom, / joint_states, without its prefix barista_robot.

File: urdf/barista_robot_model.urdf (robot description, URDF)
Before this commit: robot barista_robot, 15 links, 14 joints
Links:
- link back_pitch_link: mass 0.01 -> 0.1; geometry collision sphere radius=0.0252; visual sphere radius=0.0252
- link back_roll_link: mass 0.005 -> 0.001; geometry collision cylinder length=0.001 radius=0.0125000000000000005; visual cylinder length=0.001 radius=0.0125000000000000005
- link back_yaw_link: mass 0.005 -> 0.001; geometry collision cylinder length=0.001 radius=0.0125000000000000005; visual cylinder length=0.001 radius=0.0125000000000000005
- link front_pitch_link: mass 0.01 -> 0.1; geometry collision sphere radius=0.0252; visual sphere radius=0.0252
- link front_roll_link: mass 0.005 -> 0.001; geometry collision cylinder length=0.001 radius=0.0125000000000000005; visual cylinder length=0.001 radius=0.0125000000000000005
- link front_yaw_link: mass 0.005 -> 0.001; geometry collision cylinder length=0.001 radius=0.0125000000000000005; visual cylinder length=0.001 radius=0.0125000000000000005
- link motorized_wheel_left: geometry collision cylinder length=0.0206 radius=0.0352; visual cylinder length=0.0206 radius=0.0352
- link motorized_wheel_right: geometry collision cylinder length=0.0206 radius=0.0352; visual cylinder length=0.0206 radius=0.0352
Joints:
- joint base_to_wheel_left: origin xyz=0 0.128 -0.077 rpy=0 0 0 -> xyz=0 0.128 -0.067 rpy=0 0 0
- joint base_to_wheel_right: origin xyz=0 -0.128 -0.077 rpy=0 0 0 -> xyz=0 -0.128 -0.067 rpy=0 0 0

Commit message: Added cupholder tray link and corresponding joint. Tested in Rviz and Gazebo.

File: urdf/barista_robot_model.urdf (robot description, URDF)
Before this commit: robot barista_robot, 15 links, 14 joints
Links:
- added link cup_holder_tray, mass 2.0; collision cylinder length=0.090 radius=0.160; visual cylinder length=0.090 radius=0.160
Joints:
- added joint base_to_cup_holder_tray: type fixed, parent base_link, child cup_holder_tray, origin xyz=0 0 0.3025 rpy=0 0 0
