Commit message: Two robot spawn completed. Laser working, odom, working, no name conflicts with topic, node , tf_frames. Rick is blue, Morty is red. Rviz and Gazebo configured to show both robots.

File: xacro/cup_holder_tray.xacro (robot description, xacro)
@@ -10,5 +10,5 @@
                     <cylinder length="${cup_holder_tray_length}" radius="${cup_holder_tray_radius}"/>
                 </geometry>
-                <material name="blue"/>
+                <material name="cup_holder_tray"/>
             </visual>
             <collision>
