Commit message: Tf broadcaster improved, bugs fixed. Changed robot description files.

File: xacro/barista_multiple_robot_model.gazebo.xacro (robot description, xacro)
@@ -38,6 +38,6 @@
             <kp>1000000000000000000000000000.0</kp>
             <kd>1000000000000000000000000000.0</kd>
-            <mu1>10.0</mu1>
-            <mu2>10.0</mu2>
+            <mu1>50.0</mu1>
+            <mu2>50.0</mu2>
             <material>Gazebo/Green</material>
         </gazebo>
@@ -45,6 +45,6 @@
             <kp>1000000000000000000000000000.0</kp>
             <kd>1000000000000000000000000000.0</kd>
-            <mu1>10.0</mu1>
-            <mu2>10.0</mu2>
+            <mu1>50.0</mu1>
+            <mu2>50.0</mu2>
             <material>Gazebo/Green</material>
         </gazebo>
@@ -58,6 +58,6 @@
             <kp>1000000000000000000000000000.0</kp>
             <kd>1000000000000000000000000000.0</kd>
-            <mu1>0.5</mu1>
-            <mu2>0.5</mu2>
+            <mu1>1.5</mu1>
+            <mu2>1.5</mu2>
             <material>Gazebo/Purple</material>
         </gazebo>
@@ -71,6 +71,6 @@
             <kp>1000000000000000000000000000.0</kp>
             <kd>1000000000000000000000000000.0</kd>
-            <mu1>0.5</mu1>
-            <mu2>0.5</mu2>
+            <mu1>1.5</mu1>
+            <mu2>1.5</mu2>
             <material>Gazebo/Yellow</material>
         </gazebo>
@@ -95,5 +95,5 @@
                     <remapping>/cmd_vel:=cmd_vel</remapping>
                 </ros>
-            <update_rate>30</update_rate>
+            <update_rate>50</update_rate>
             <!-- wheels -->
             <left_joint>base_to_wheel_left</left_joint>
@@ -106,9 +106,9 @@
             <odometry_frame>${robot_name}/odom</odometry_frame>
             <robot_base_frame>${robot_name}/base_link</robot_base_frame>
-            <publish_odom_tf>true</publish_odom_tf>
+            <publish_odom_tf>false</publish_odom_tf>
             <publish_wheel_tf>false</publish_wheel_tf>
             <!-- limits -->
-            <max_wheel_torque>1.0</max_wheel_torque>
-            <max_wheel_acceleration>2.0</max_wheel_acceleration>
+            <max_wheel_torque>10.0</max_wheel_torque>
+            <max_wheel_acceleration>5.0</max_wheel_acceleration>
             </plugin>
         </gazebo>

File: xacro/barista_multiple_robot_model.urdf.xacro (robot description, xacro)
@@ -188,6 +188,6 @@
         <origin rpy="0 0 0" xyz="0 0.128 -0.067"/>
         <axis xyz="0 1 0"/>
-        <limit effort="1.0" velocity="10.0"/>
-        <dynamics damping="0.1" friction="0.1"/>
+        <limit effort="10000" velocity="1000"/>
+        <dynamics damping="1.0" friction="1.0"/>
     </joint>
     <joint name="base_to_wheel_right" type="continuous">
@@ -196,6 +196,6 @@
         <origin rpy="0 0 0" xyz="0 -0.128 -0.067"/>
         <axis xyz="0 1 0"/>
-        <limit effort="1.0" velocity="10.0"/>
-        <dynamics damping="0.1" friction="0.1"/>
+        <limit effort="10000" velocity="1000"/>
+        <dynamics damping="1.0" friction="1.0"/>
     </joint>
     <!-- Caster Wheels -->

Commit message: Files edited to make it work with robot_chase.

File: xacro/barista_multiple_robot_model.gazebo.xacro (robot description, xacro)
@@ -38,6 +38,6 @@
             <kp>1000000000000000000000000000.0</kp>
             <kd>1000000000000000000000000000.0</kd>
-            <mu1>50.0</mu1>
-            <mu2>50.0</mu2>
+            <mu1>100.0</mu1>
+            <mu2>100.0</mu2>
             <material>Gazebo/Green</material>
         </gazebo>
@@ -45,6 +45,6 @@
             <kp>1000000000000000000000000000.0</kp>
             <kd>1000000000000000000000000000.0</kd>
-            <mu1>50.0</mu1>
-            <mu2>50.0</mu2>
+            <mu1>100.0</mu1>
+            <mu2>100.0</mu2>
             <material>Gazebo/Green</material>
         </gazebo>
@@ -95,5 +95,5 @@
                     <remapping>/cmd_vel:=cmd_vel</remapping>
                 </ros>
-            <update_rate>50</update_rate>
+            <update_rate>50.0</update_rate>
             <!-- wheels -->
             <left_joint>base_to_wheel_left</left_joint>
@@ -109,6 +109,6 @@
             <publish_wheel_tf>false</publish_wheel_tf>
             <!-- limits -->
-            <max_wheel_torque>10.0</max_wheel_torque>
-            <max_wheel_acceleration>5.0</max_wheel_acceleration>
+            <max_wheel_torque>7.0</max_wheel_torque>
+            <max_wheel_acceleration>2.0</max_wheel_acceleration>
             </plugin>
         </gazebo>
@@ -175,5 +175,5 @@
                     <always_on>true</always_on>
                     <visualize>true</visualize>
-                    <update_rate>30.0</update_rate>
+                    <update_rate>50.0</update_rate>
                     <plugin name="laser" filename="libgazebo_ros_ray_sensor.so">
                         <ros>
@@ -195,5 +195,5 @@
                     <remapping>~/out:=joint_states</remapping>
                 </ros>
-                <update_rate>30</update_rate>
+                <update_rate>50.0</update_rate>
                 <joint_name>base_to_wheel_left</joint_name>
                 <joint_name>base_to_wheel_right</joint_name>

File: xacro/barista_multiple_robot_model.urdf.xacro (robot description, xacro)
@@ -189,5 +189,5 @@
         <axis xyz="0 1 0"/>
         <limit effort="10000" velocity="1000"/>
-        <dynamics damping="1.0" friction="1.0"/>
+        <dynamics damping="1.0" friction="3.0"/>
     </joint>
     <joint name="base_to_wheel_right" type="continuous">
@@ -197,5 +197,5 @@
         <axis xyz="0 1 0"/>
         <limit effort="10000" velocity="1000"/>
-        <dynamics damping="1.0" friction="1.0"/>
+        <dynamics damping="1.0" friction="3.0"/>
     </joint>
     <!-- Caster Wheels -->

Commit message: Fixed torque and acceleration errors. Robot can now have a linear and angular velocity at the same time and make circular movements. the robot can also stop and act quicker to /cmd_vel pubs. base wheel left and right joint attributes changed.

File: xacro/barista_multiple_robot_model.gazebo.xacro (robot description, xacro)
@@ -109,6 +109,6 @@
             <publish_wheel_tf>false</publish_wheel_tf>
             <!-- limits -->
-            <max_wheel_torque>7.0</max_wheel_torque>
-            <max_wheel_acceleration>2.0</max_wheel_acceleration>
+        <max_wheel_torque>4.0</max_wheel_torque>
+        <max_wheel_acceleration>4.0</max_wheel_acceleration>
             </plugin>
         </gazebo>
@@ -204,6 +204,4 @@
                 <joint_name>front_pitch_joint</joint_name>
                 <joint_name>back_pitch_joint</joint_name>
-                <joint_name>laser_scan_link_joint</joint_name>
-                <joint_name>laser_scan_frame_joint</joint_name>
             </plugin>
         </gazebo>

File: xacro/barista_multiple_robot_model.urdf.xacro (robot description, xacro)
@@ -188,6 +188,6 @@
         <origin rpy="0 0 0" xyz="0 0.128 -0.067"/>
         <axis xyz="0 1 0"/>
-        <limit effort="10000" velocity="1000"/>
-        <dynamics damping="1.0" friction="3.0"/>
+        <limit effort="1.0" velocity="10.0"/>
+        <dynamics damping="0.1" friction="0.1"/>
     </joint>
     <joint name="base_to_wheel_right" type="continuous">
@@ -196,6 +196,6 @@
         <origin rpy="0 0 0" xyz="0 -0.128 -0.067"/>
         <axis xyz="0 1 0"/>
-        <limit effort="10000" velocity="1000"/>
-        <dynamics damping="1.0" friction="3.0"/>
+        <limit effort="1.0" velocity="10.0"/>
+        <dynamics damping="0.1" friction="0.1"/>
     </joint>
     <!-- Caster Wheels -->

File: xacro/barista_robot_model.urdf.xacro (robot description, xacro)
@@ -356,8 +356,8 @@
         <!-- kinematics -->
         <wheel_separation>0.256</wheel_separation>
-        <wheel_diameter>0.06</wheel_diameter>
+        <wheel_diameter>0.0704</wheel_diameter>
         <!-- limits -->
-        <max_wheel_torque>1.0</max_wheel_torque>
-        <max_wheel_acceleration>2.0</max_wheel_acceleration>
+        <max_wheel_torque>4.0</max_wheel_torque>
+        <max_wheel_acceleration>4.0</max_wheel_acceleration>
         <!-- output -->
         <publish_odom>true</publish_odom>
